Commit message: Update urdf files

File: akabot_description/urdf/akabot.ros2_control.xacro (robot description, xacro)
@@ -1,112 +1,68 @@
 <?xml version="1.0"?>
 <robot xmlns:xacro="http://www.ros.org/wiki/xacro">
-    <xacro:property name="initial_positions" value="${load_yaml(initial_positions_file)['initial_positions']}"/>
-      <!-- Gazebo ros2_control -->
-      <xacro:if value="$(arg sim_mode)"
-        <ros2_control name="GazeboSystem" type="system">
-            <hardware>
-                <plugin>gazebo_ros2_control/GazeboSystem</plugin>
-            </hardware>
-            <joint name="right_claw_joint">
-                <command_interface name="position"/>
-                <state_interface name="position">
-                  <param name="initial_value">${initial_positions['right_claw_joint']}</param>
-                </state_interface>
-                <state_interface name="velocity"/>
-            </joint>
-            <joint name="top_plate_joint">
-                <command_interface name="position"/>
-                <state_interface name="position">
-                  <param name="initial_value">${initial_positions['top_plate_joint']}</param>
-                </state_interface>
-                <state_interface name="velocity"/>
-            </joint>
-            <joint name="lower_arm_joint">
-                <command_interface name="position"/>
-                <state_interface name="position">
-                  <param name="initial_value">${initial_positions['lower_arm_joint']}</param>
-                </state_interface>
-                <state_interface name="velocity"/>
-            </joint>
-            <joint name="upper_arm_joint">
-                <command_interface name="position"/>
-                <state_interface name="position">
-                  <param name="initial_value">${initial_positions['upper_arm_joint']}</param>
-                </state_interface>
-                <state_interface name="velocity"/>
-            </joint>
-            <joint name="wrist_joint">
-                <command_interface name="position"/>
-                <state_interface name="position">
-                  <param name="initial_value">${initial_positions['wrist_joint']}</param>
-                </state_interface>
-                <state_interface name="velocity"/>
-            </joint>
-            <joint name="claw_base_joint">
-                <command_interface name="position"/>
-                <state_interface name="position">
-                  <param name="initial_value">${initial_positions['claw_base_joint']}</param>
-                </state_interface>
-                <state_interface name="velocity"/>
-            </joint>
-        </ros2_control>
-      </xacro:if>
-    <gazebo>
-      <plugin name="gazebo_ros2_control" filename="libgazebo_ros2_control.so">
-        <parameters>$(find akabot_moveit_config)/config/ros2_controllers.yaml</parameters>
-      </plugin>
-    </gazebo>
-    <!-- Mock components -->
-    <xacro:macro name="akabot_ros2_control" params="name initial_positions_file">
-      <xacro:if value="$(arg use_mock)"
-        <ros2_control name="${name}" type="system">
-            <hardware>
-                <!-- By default, set up controllers for simulation. This won't work on real hardware -->
-                <plugin>mock_components/GenericSystem</plugin>
-            </hardware>
-            <joint name="right_claw_joint">
-                <command_interface name="position"/>
-                <state_interface name="position">
-                  <param name="initial_value">${initial_positions['right_claw_joint']}</param>
-                </state_interface>
-                <state_interface name="velocity"/>
-            </joint>
-            <joint name="top_plate_joint">
-                <command_interface name="position"/>
-                <state_interface name="position">
-                  <param name="initial_value">${initial_positions['top_plate_joint']}</param>
-                </state_interface>
-                <state_interface name="velocity"/>
-            </joint>
-            <joint name="lower_arm_joint">
-                <command_interface name="position"/>
-                <state_interface name="position">
-                  <param name="initial_value">${initial_positions['lower_arm_joint']}</param>
-                </state_interface>
-                <state_interface name="velocity"/>
-            </joint>
-            <joint name="upper_arm_joint">
-                <command_interface name="position"/>
-                <state_interface name="position">
-                  <param name="initial_value">${initial_positions['upper_arm_joint']}</param>
-                </state_interface>
-                <state_interface name="velocity"/>
-            </joint>
-            <joint name="wrist_joint">
-                <command_interface name="position"/>
-                <state_interface name="position">
-                  <param name="initial_value">${initial_positions['wrist_joint']}</param>
-                </state_interface>
-                <state_interface name="velocity"/>
-            </joint>
-            <joint name="claw_base_joint">
-                <command_interface name="position"/>
-                <state_interface name="position">
-                  <param name="initial_value">${initial_positions['claw_base_joint']}</param>
-                </state_interface>
-                <state_interface name="velocity"/>
-            </joint>
-        </ros2_control>
-      </xacro:if>
-    </xacro:macro>
+  <!-- Properties -->
+  <xacro:property name="initial_positions_file" value="$(find akabot_description)/config/initial_positions.yaml"/>
+  <xacro:property name="initial_positions" value="${load_yaml(initial_positions_file)['initial_positions']}"/>
+  <!-- ros2_control macro -->
+  <xacro:macro name="akabot_ros2_control" params="name plugin_name">
+    <ros2_control name="${name}" type="system">
+      <hardware>
+        <plugin>${plugin_name}</plugin>
+      </hardware>
+      <joint name="right_claw_joint">
+        <command_interface name="position"/>
+          <param name="min">-0.5</param>
+          <param name="max">0.0</param>
+        <state_interface name="position">
+          <param name="initial_value">${initial_positions['right_claw_joint']}</param>
+        </state_interface>
+        <state_interface name="velocity"/>
+      </joint>
+      <joint name="top_plate_joint">
+        <command_interface name="position"/>
+          <param name="min">1.56</param>
+          <param name="max">4.68</param>
+        <state_interface name="position">
+          <param name="initial_value">${initial_positions['top_plate_joint']}</param>
+        </state_interface>
+        <state_interface name="velocity"/>
+      </joint>
+      <joint name="lower_arm_joint">
+        <command_interface name="position"/>
+          <param name="min">0.0</param>
+          <param name="max">3.12</param>
+        <state_interface name="position">
+          <param name="initial_value">${initial_positions['lower_arm_joint']}</param>
+        </state_interface>
+        <state_interface name="velocity"/>
+      </joint>
+      <joint name="upper_arm_joint">
+        <command_interface name="position"/>
+          <param name="min">-1.7</param>
+          <param name="max">1.7</param>
+        <state_interface name="position">
+          <param name="initial_value">${initial_positions['upper_arm_joint']}</param>
+        </state_interface>
+        <state_interface name="velocity"/>
+      </joint>
+      <joint name="wrist_joint">
+        <command_interface name="position"/>
+          <param name="min">-1.7</param>
+          <param name="max">1.7</param>
+        <state_interface name="position">
+          <param name="initial_value">${initial_positions['wrist_joint']}</param>
+        </state_interface>
+        <state_interface name="velocity"/>
+      </joint>
+      <joint name="claw_base_joint">
+        <command_interface name="position"/>
+          <param name="min">-3.17</param>
+          <param name="max">0.0</param>
+        <state_interface name="position">
+          <param name="initial_value">${initial_positions['claw_base_joint']}</param>
+        </state_interface>
+        <state_interface name="velocity"/>
+      </joint>
+    </ros2_control>
+  </xacro:macro>
 </robot>

File: akabot_description/urdf/akabot.urdf.xacro (robot description, xacro)
@@ -1,7 +1,5 @@
 <?xml version="1.0" ?>
 <robot name="akabot" xmlns:xacro="http://ros.org/wiki/xacro">
-    <xacro:arg name="sim_mode" default="false">
     <xacro:include filename="akabot_core.xacro"/>
     <xacro:include filename="depth_camera.xacro"/>
-    <xacro:include filename="ros2_control.xacro"/>
 </robot>

File: akabot_moveit_config/urdf/fake.akabot.urdf.xacro (robot description, xacro)
@@ -1,9 +1,8 @@
 <?xml version="1.0"?>
 <robot xmlns:xacro="http://www.ros.org/wiki/xacro" name="akabot">
-    <xacro:arg name="initial_positions_file" default="initial_positions.yaml" />
-    <!-- Import akabot urdf file -->
-    <xacro:include filename="$(find akabot_description)/urdf/akabot.urdf.xacro" />
-    <!-- Import control_xacro -->
-    <xacro:include filename="$(find akabot_description)/urdf/akabot.ros2_control.xacro" />
-    <xacro:akabot_ros2_control name="FakeSystem" initial_positions_file="$(arg initial_positions_file)"/>
+    <!-- Import akabot urdf and ros2_control xacro files -->
+    <xacro:include filename="$(find akabot_description)/urdf/akabot.urdf.xacro"/>
+    <xacro:include filename="$(find akabot_description)/urdf/akabot.ros2_control.xacro"/>
+    <!-- ros2_control macro -->
+    <xacro:akabot_ros2_control name="FakeSystem" plugin_name="mock_components/GenericSystem"/>
 </robot>

Commit message: Configure akabot hand/gripper planning group to work in Moveit

File: akabot_description/urdf/akabot.ros2_control.xacro (robot description, xacro)
@@ -3,5 +3,5 @@
   <!-- Properties -->
   <xacro:property name="initial_positions_file" value="$(find akabot_description)/config/initial_positions.yaml"/>
-  <xacro:property name="initial_positions" value="${load_yaml(initial_positions_file)['initial_positions']}"/>
+  <xacro:property name="initial_positions" value="${xacro.load_yaml(initial_positions_file)['initial_positions']}"/>
   <!-- ros2_control macro -->
   <xacro:macro name="akabot_ros2_control" params="name plugin_name">
@@ -64,4 +64,24 @@
         <state_interface name="velocity"/>
       </joint>
+      <joint name="right_claw_joint">
+        <command_interface name="position"/>
+          <param name="min">-0.5</param>
+          <param name="max">0.0</param>
+        <state_interface name="position">
+          <param name="initial_value">${initial_positions['right_claw_joint']}</param>
+        </state_interface>
+        <state_interface name="velocity"/>
+      </joint>
+      <joint name="left_claw_joint">
+        <param name="mimic">right_claw_joint</param>
+        <param name="multiplier">-1</param>
+        <command_interface name="position"/>
+          <param name="min">0.0</param>
+          <param name="max">0.5</param>
+        <state_interface name="position">
+          <param name="initial_value">${initial_positions['left_claw_joint']}</param>
+        </state_interface>
+        <state_interface name="velocity"/>
+      </joint>
     </ros2_control>
   </xacro:macro>

File: akabot_description/urdf/akabot_core.xacro (robot description, xacro)
@@ -187,5 +187,5 @@
     <origin rpy="0 0 0.22" xyz="-0.16 0.30 0"/>
     <axis xyz="0 0 1" />
-    <limit effort="1000.0" lower="0" upper="-0.5" velocity="1.0" />
+    <limit effort="1000.0" lower="0.0" upper="0.5" velocity="1.0" />
     <mimic joint="right_claw_joint" multiplier="-1" offset="0" />
   </joint>

Commit message: Fix gripper action in Gazebo

File: akabot_description/urdf/akabot.ros2_control.xacro (robot description, xacro)
@@ -10,13 +10,4 @@
         <plugin>${plugin_name}</plugin>
       </hardware>
-      <joint name="right_claw_joint">
-        <command_interface name="position"/>
-          <param name="min">-0.5</param>
-          <param name="max">0.0</param>
-        <state_interface name="position">
-          <param name="initial_value">${initial_positions['right_claw_joint']}</param>
-        </state_interface>
-        <state_interface name="velocity"/>
-      </joint>
       <joint name="top_plate_joint">
         <command_interface name="position"/>

File: akabot_description/urdf/depth_camera.xacro (robot description, xacro)
@@ -8,5 +8,5 @@
         </geometry>
     </visual>
- 	  <collision>
+    <collision>
       <origin xyz="0.4 -0.015 0.135" rpy="${-pi/2} ${pi} ${-pi/2}"/>
         <geometry>
@@ -32,19 +32,19 @@
         <update_rate>10</update_rate>
         <camera>
-          <horizontal_fov>1.134</horizontal_fov>
+          <horizontal_fov>1.2113</horizontal_fov>
           <image>
-              <format>B8G8R8</format>
-              <width>640</width>
-              <height>480</height>
+            <format>B8G8R8</format>
+            <width>1280</width>
+            <height>720</height>
           </image>
           <clip>
-              <near>0.05</near>
-              <far>8.0</far>
+            <near>0.05</near>
+            <far>8.0</far>
           </clip>
         </camera>
         <plugin name="camera_controller" filename="libgazebo_ros_camera.so">
-            <frame_name>camera_link_optical</frame_name>
-            <min_depth>0.1</min_depth>
-            <max_depth>100.0</max_depth>
+          <frame_name>camera_link_optical</frame_name>
+          <min_depth>0.1</min_depth>
+          <max_depth>100.0</max_depth>
         </plugin>
     </sensor>
