Commit message: Add placeholder inertia values in akabot_core.xacro

File: akabot_description/urdf/akabot_core.xacro (robot description, xacro)
@@ -14,4 +14,5 @@
         <geometry>
           <mesh filename="package://akabot_description/meshes/base_cylinder.stl" scale ="0.0001 0.0001 0.0001"/>
+          <!-- <mesh filename="file://$(find akabot_description)/meshes/base_cylinder.stl" scale ="0.0001 0.0001 0.0001"/> -->
         </geometry>
         <material name="black">
@@ -23,6 +24,17 @@
         <geometry>
           <mesh filename="package://akabot_description/meshes/base_cylinder.stl" scale ="0.0001 0.0001 0.0001"/>
+          <!-- <mesh filename="file://$(find akabot_description)/meshes/base_cylinder.stl" scale ="0.0001 0.0001 0.0001"/> -->
         </geometry>
     </collision>
+		<inertial>
+      <mass value="0.540142"/>
+      <inertia
+        ixx="0.0021190000"
+        iyy="0.0006925000"
+        izz="0.0025280000"
+        ixy="-0.0000172100"
+        ixz="0.0000006389"
+        iyz="0.0000461200"/>
+    </inertial>
   </link>
   <joint name="top_plate_joint" type="revolute">
@@ -39,4 +51,5 @@
         <geometry>
           <mesh filename="package://akabot_description/meshes/top_plate.stl" scale ="0.001 0.001 0.001"/>
+          <!-- <mesh filename="file://$(find akabot_description)/meshes/top_plate.stl" scale ="0.001 0.001 0.001"/> -->
         </geometry>
         <material name="black"/>
@@ -46,6 +59,17 @@
       <geometry>
         <mesh filename="package://akabot_description/meshes/top_plate.stl" scale ="0.001 0.001 0.001"/>
-      </geometry>
-        </collision>
+        <!-- <mesh filename="file://$(find akabot_description)/meshes/top_plate.stl" scale ="0.001 0.001 0.001"/> -->
+      </geometry>
+    </collision>
+		<inertial>
+      <mass value="0.480879"/>
+      <inertia
+        ixx="0.0003790000"
+        iyy="0.0005557000"
+        izz="0.0005889000"
+        ixy="0.0000000022"
+        ixz="-0.0000003561"
+        iyz="0.0000012247"/>
+		</inertial>
   </link>
   <joint name="lower_arm_joint" type="revolute">
@@ -62,4 +86,5 @@
       <geometry>
         <mesh filename="package://akabot_description/meshes/lower_arm.stl" scale ="0.001 0.001 0.001"/>
+        <!-- <mesh filename="file://$(find akabot_description)/meshes/lower_arm.stl" scale ="0.001 0.001 0.001"/> -->
       </geometry>
       <material name="black"/>
@@ -69,6 +94,17 @@
       <geometry>
         <mesh filename="package://akabot_description/meshes/lower_arm.stl" scale ="0.001 0.001 0.001"/>
-      </geometry>
-    </collision>
+        <!-- <mesh filename="file://$(find akabot_description)/meshes/lower_arm.stl" scale ="0.001 0.001 0.001"/> -->
+      </geometry>
+    </collision>
+		<inertial>
+      <mass value="0.297781"/>
+      <inertia
+        ixx="0.0017100000"
+        iyy="0.0016310000"
+        izz="0.0001482000"
+        ixy="-0.0000011433"
+        ixz="0.0000021161"
+        iyz="0.0002135000"/>
+    </inertial>
   </link>
   <joint name="upper_arm_joint" type="revolute">
@@ -85,4 +121,5 @@
       <geometry>
         <mesh filename="package://akabot_description/meshes/upper_arm.stl" scale ="0.001 0.001 0.001"/>
+        <!-- <mesh filename="file://$(find akabot_description)/meshes/upper_arm.stl" scale ="0.001 0.001 0.001"/> -->
       </geometry>
       <material name="black"/>
@@ -92,6 +129,11 @@
       <geometry>
         <mesh filename="package://akabot_description/meshes/upper_arm.stl" scale ="0.001 0.001 0.001"/>
-      </geometry>
-    </collision>
+        <!-- <mesh filename="file://$(find akabot_description)/meshes/upper_arm.stl" scale ="0.001 0.001 0.001"/> -->
+      </geometry>
+    </collision>
+		<inertial>
+			<mass value="2e-06"/>
+			<inertia ixx="1.1e-09" ixy="0" ixz="0" iyy="1.1e-09" iyz="0" izz="1.1e-09"/>
+		</inertial>
   </link>
   <joint name="wrist_joint" type="revolute">
@@ -108,4 +150,5 @@
       <geometry>
         <mesh filename="package://akabot_description/meshes/wrist.stl" scale ="0.001 0.001 0.001"/>
+        <!-- <mesh filename="file://$(find akabot_description)/meshes/wrist.stl" scale ="0.001 0.001 0.001"/> -->
       </geometry>
       <material name="black"/>
@@ -115,6 +158,17 @@
       <geometry>
         <mesh filename="package://akabot_description/meshes/wrist.stl" scale ="0.001 0.001 0.001"/>
-      </geometry>
-    </collision>
+        <!-- <mesh filename="file://$(find akabot_description)/meshes/wrist.stl" scale ="0.001 0.001 0.001"/> -->
+      </geometry>
+    </collision>
+		<inertial>
+      <mass value="0.283651"/>
+      <inertia
+        ixx="0.0011850000"
+        iyy="0.0000682900"
+        izz="0.0012060000"
+        ixy="-0.0000024317"
+        ixz="0.0000000000"
+        iyz="0.0000000000"/>
+    </inertial>
   </link>
   <joint name="claw_base_joint" type="revolute">
@@ -131,4 +185,5 @@
       <geometry>
         <mesh filename="package://akabot_description/meshes/claw_base.stl" scale ="0.001 0.001 0.001"/>
+        <!-- <mesh filename="file://$(find akabot_description)/meshes/claw_base.stl" scale ="0.001 0.001 0.001"/> -->
       </geometry>
       <material name="white">
@@ -140,6 +195,17 @@
       <geometry>
         <mesh filename="package://akabot_description/meshes/claw_base.stl" scale ="0.001 0.001 0.001"/>
-      </geometry>
-    </collision>
+        <!-- <mesh filename="file://$(find akabot_description)/meshes/claw_base.stl" scale ="0.001 0.001 0.001"/> -->
+      </geometry>
+    </collision>
+		<inertial>
+     <mass value="0.084957"/>
+      <inertia
+        ixx="0.0000308200"
+        iyy="0.0000282200"
+        izz="0.0000315200"
+        ixy="0.0000000191"
+        ixz="0.0000000023"
+        iyz="0.0000025481"/>
+    </inertial>
   </link>
   <joint name="right_claw_joint" type="revolute">
@@ -156,4 +222,5 @@
       <geometry>
         <mesh filename="package://akabot_description/meshes/right_claw.stl" scale ="0.001 0.001 0.001"/>
+        <!-- <mesh filename="file://$(find akabot_description)/meshes/right_claw.stl" scale ="0.001 0.001 0.001"/> -->
       </geometry>
       <material name="white"/>
@@ -163,6 +230,17 @@
       <geometry>
         <mesh filename="package://akabot_description/meshes/right_claw.stl" scale ="0.001 0.001 0.001"/>
-      </geometry>
-    </collision>
+        <!-- <mesh filename="file://$(find akabot_description)/meshes/right_claw.stl" scale ="0.001 0.001 0.001"/> -->
+      </geometry>
+    </collision>
+		<inertial>
+      <mass value="0.072885"/>
+      <inertia
+        ixx="0.0000253700"
+        iyy="0.0000183600"
+        izz="0.0000167400"
+        ixy="0.0000000000"
+        ixz="0.0000000000"
+        iyz="0.0000004340"/>
+      </inertial>
   </link>
   <!-- Left claw -->
@@ -172,4 +250,5 @@
       <geometry>
         <mesh filename="package://akabot_description/meshes/left_claw.stl" scale ="0.001 0.001 0.001"/>
+        <!-- <mesh filename="file://$(find akabot_description)/meshes/left_claw.stl" scale ="0.001 0.001 0.001"/> -->
       </geometry>
       <material name="white"/>
@@ -179,6 +258,17 @@
       <geometry>
         <mesh filename="package://akabot_description/meshes/left_claw.stl" scale ="0.001 0.001 0.001"/>
-      </geometry>
-    </collision>
+        <!-- <mesh filename="file://$(find akabot_description)/meshes/left_claw.stl" scale ="0.001 0.001 0.001"/> -->
+      </geometry>
+    </collision>
+		<inertial>
+      <mass value="0.072885"/>
+      <inertia
+        ixx="0.0000253700"
+        iyy="0.0000183600"
+        izz="0.0000167400"
+        ixy="0.0000000000"
+        ixz="0.0000000000"
+        iyz="0.0000004340"/>
+    </inertial>
   </link>
   <joint name="left_claw_joint" type="revolute">

Commit message: Update akabot initial positions

File: akabot_description/urdf/akabot_core.xacro (robot description, xacro)
@@ -13,5 +13,6 @@
       <origin xyz="0 0 0.01"/>
         <geometry>
-          <mesh filename="package://akabot_description/meshes/base_cylinder.stl" scale ="0.0001 0.0001 0.0001"/>
+          <mesh filename="package://akabot_description/meshes/base_cylinder.dae"/>
+          <!-- <mesh filename="package://akabot_description/meshes/base_cylinder.stl" scale ="0.0001 0.0001 0.0001"/> -->
           <!-- <mesh filename="file://$(find akabot_description)/meshes/base_cylinder.stl" scale ="0.0001 0.0001 0.0001"/> -->
         </geometry>
@@ -23,5 +24,6 @@
       <origin xyz="0 0 0.01"/>
         <geometry>
-          <mesh filename="package://akabot_description/meshes/base_cylinder.stl" scale ="0.0001 0.0001 0.0001"/>
+          <mesh filename="package://akabot_description/meshes/base_cylinder.dae"/>
+          <!-- <mesh filename="package://akabot_description/meshes/base_cylinder.stl" scale ="0.0001 0.0001 0.0001"/> -->
           <!-- <mesh filename="file://$(find akabot_description)/meshes/base_cylinder.stl" scale ="0.0001 0.0001 0.0001"/> -->
         </geometry>
@@ -50,5 +52,6 @@
       <origin xyz="0 0 0"/>
         <geometry>
-          <mesh filename="package://akabot_description/meshes/top_plate.stl" scale ="0.001 0.001 0.001"/>
+          <mesh filename="package://akabot_description/meshes/top_plate.dae"/>
+          <!-- <mesh filename="package://akabot_description/meshes/top_plate.stl" scale ="0.001 0.001 0.001"/> -->
           <!-- <mesh filename="file://$(find akabot_description)/meshes/top_plate.stl" scale ="0.001 0.001 0.001"/> -->
         </geometry>
@@ -58,5 +61,6 @@
       <!-- <origin xyz="0 0 0"/> -->
       <geometry>
-        <mesh filename="package://akabot_description/meshes/top_plate.stl" scale ="0.001 0.001 0.001"/>
+        <mesh filename="package://akabot_description/meshes/top_plate.dae"/>
+        <!-- <mesh filename="package://akabot_description/meshes/top_plate.stl" scale ="0.001 0.001 0.001"/> -->
         <!-- <mesh filename="file://$(find akabot_description)/meshes/top_plate.stl" scale ="0.001 0.001 0.001"/> -->
       </geometry>
@@ -85,5 +89,6 @@
       <!-- <origin xyz="0 0 0"/> -->
       <geometry>
-        <mesh filename="package://akabot_description/meshes/lower_arm.stl" scale ="0.001 0.001 0.001"/>
+        <mesh filename="package://akabot_description/meshes/lower_arm.dae"/>
+        <!-- <mesh filename="package://akabot_description/meshes/lower_arm.stl" scale ="0.001 0.001 0.001"/> -->
         <!-- <mesh filename="file://$(find akabot_description)/meshes/lower_arm.stl" scale ="0.001 0.001 0.001"/> -->
       </geometry>
@@ -93,5 +98,6 @@
       <origin xyz="0 0 0"/>
       <geometry>
-        <mesh filename="package://akabot_description/meshes/lower_arm.stl" scale ="0.001 0.001 0.001"/>
+        <mesh filename="package://akabot_description/meshes/lower_arm.dae"/>
+        <!-- <mesh filename="package://akabot_description/meshes/lower_arm.stl" scale ="0.001 0.001 0.001"/> -->
         <!-- <mesh filename="file://$(find akabot_description)/meshes/lower_arm.stl" scale ="0.001 0.001 0.001"/> -->
       </geometry>
@@ -120,5 +126,6 @@
       <origin rpy="0 1.59 0" xyz="0 0 0"/>
       <geometry>
-        <mesh filename="package://akabot_description/meshes/upper_arm.stl" scale ="0.001 0.001 0.001"/>
+        <mesh filename="package://akabot_description/meshes/upper_arm.dae"/>
+        <!-- <mesh filename="package://akabot_description/meshes/upper_arm.stl" scale ="0.001 0.001 0.001"/> -->
         <!-- <mesh filename="file://$(find akabot_description)/meshes/upper_arm.stl" scale ="0.001 0.001 0.001"/> -->
       </geometry>
@@ -128,5 +135,6 @@
       <origin rpy="0 1.59 0" xyz="0 0 0"/>
       <geometry>
-        <mesh filename="package://akabot_description/meshes/upper_arm.stl" scale ="0.001 0.001 0.001"/>
+        <mesh filename="package://akabot_description/meshes/upper_arm.dae"/>
+        <!-- <mesh filename="package://akabot_description/meshes/upper_arm.stl" scale ="0.001 0.001 0.001"/> -->
         <!-- <mesh filename="file://$(find akabot_description)/meshes/upper_arm.stl" scale ="0.001 0.001 0.001"/> -->
       </geometry>
@@ -149,5 +157,6 @@
       <!-- <origin rpy="0 0 0" xyz="0 0 0"/> -->
       <geometry>
-        <mesh filename="package://akabot_description/meshes/wrist.stl" scale ="0.001 0.001 0.001"/>
+        <mesh filename="package://akabot_description/meshes/wrist.dae"/>
+        <!-- <mesh filename="package://akabot_description/meshes/wrist.stl" scale ="0.001 0.001 0.001"/> -->
         <!-- <mesh filename="file://$(find akabot_description)/meshes/wrist.stl" scale ="0.001 0.001 0.001"/> -->
       </geometry>
@@ -157,5 +166,6 @@
       <origin rpy="0 0 0" xyz="0 0 0"/>
       <geometry>
-        <mesh filename="package://akabot_description/meshes/wrist.stl" scale ="0.001 0.001 0.001"/>
+        <mesh filename="package://akabot_description/meshes/wrist.dae"/>
+        <!-- <mesh filename="package://akabot_description/meshes/wrist.stl" scale ="0.001 0.001 0.001"/> -->
         <!-- <mesh filename="file://$(find akabot_description)/meshes/wrist.stl" scale ="0.001 0.001 0.001"/> -->
       </geometry>
@@ -184,5 +194,6 @@
       <origin rpy="0 3.18 0" xyz="0 0 0"/>
       <geometry>
-        <mesh filename="package://akabot_description/meshes/claw_base.stl" scale ="0.001 0.001 0.001"/>
+        <mesh filename="package://akabot_description/meshes/claw_base.dae"/>
+        <!-- <mesh filename="package://akabot_description/meshes/claw_base.stl" scale ="0.001 0.001 0.001"/> -->
         <!-- <mesh filename="file://$(find akabot_description)/meshes/claw_base.stl" scale ="0.001 0.001 0.001"/> -->
       </geometry>
@@ -194,5 +205,6 @@
       <origin rpy="0 3.18 0" xyz="0 0 0"/>
       <geometry>
-        <mesh filename="package://akabot_description/meshes/claw_base.stl" scale ="0.001 0.001 0.001"/>
+        <mesh filename="package://akabot_description/meshes/claw_base.dae"/>
+        <!-- <mesh filename="package://akabot_description/meshes/claw_base.stl" scale ="0.001 0.001 0.001"/> -->
         <!-- <mesh filename="file://$(find akabot_description)/meshes/claw_base.stl" scale ="0.001 0.001 0.001"/> -->
       </geometry>
@@ -221,5 +233,6 @@
       <origin rpy="0 0 0" xyz="0 0 0"/>
       <geometry>
-        <mesh filename="package://akabot_description/meshes/right_claw.stl" scale ="0.001 0.001 0.001"/>
+        <mesh filename="package://akabot_description/meshes/right_claw.dae"/>
+        <!-- <mesh filename="package://akabot_description/meshes/right_claw.stl" scale ="0.001 0.001 0.001"/> -->
         <!-- <mesh filename="file://$(find akabot_description)/meshes/right_claw.stl" scale ="0.001 0.001 0.001"/> -->
       </geometry>
@@ -229,5 +242,6 @@
       <origin rpy="0 0 0" xyz="0 0 0"/>
       <geometry>
-        <mesh filename="package://akabot_description/meshes/right_claw.stl" scale ="0.001 0.001 0.001"/>
+        <mesh filename="package://akabot_description/meshes/right_claw.dae"/>
+        <!-- <mesh filename="package://akabot_description/meshes/right_claw.stl" scale ="0.001 0.001 0.001"/> -->
         <!-- <mesh filename="file://$(find akabot_description)/meshes/right_claw.stl" scale ="0.001 0.001 0.001"/> -->
       </geometry>
@@ -249,5 +263,6 @@
       <origin rpy="0 0 0" xyz="0 0 0"/>
       <geometry>
-        <mesh filename="package://akabot_description/meshes/left_claw.stl" scale ="0.001 0.001 0.001"/>
+        <mesh filename="package://akabot_description/meshes/left_claw.dae"/>
+        <!-- <mesh filename="package://akabot_description/meshes/left_claw.stl" scale ="0.001 0.001 0.001"/> -->
         <!-- <mesh filename="file://$(find akabot_description)/meshes/left_claw.stl" scale ="0.001 0.001 0.001"/> -->
       </geometry>
@@ -257,5 +272,6 @@
       <origin rpy="0 0 0" xyz="0 0 0"/>
       <geometry>
-        <mesh filename="package://akabot_description/meshes/left_claw.stl" scale ="0.001 0.001 0.001"/>
+        <mesh filename="package://akabot_description/meshes/left_claw.dae"/>
+        <!-- <mesh filename="package://akabot_description/meshes/left_claw.stl" scale ="0.001 0.001 0.001"/> -->
         <!-- <mesh filename="file://$(find akabot_description)/meshes/left_claw.stl" scale ="0.001 0.001 0.001"/> -->
       </geometry>
