Commit message: Add correct inertia values and update README

File: akabot_description/urdf/akabot_core.xacro (robot description, xacro)
@@ -1,4 +1,12 @@
 <?xml version="1.0" ?>
 <robot xmlns:xacro="http://ros.org/wiki/xacro">
+  <xacro:include filename="inertial_macros.xacro"/>
+  <!-- World link -->
+  <link name="world"/>
+  <!-- Fix base_link to Gazebo world -->
+  <joint name="fixed" type="fixed">
+    <parent link="world"/>
+    <child link="base_link"/>
+  </joint>
   <!-- Base link  -->
   <link name="base_link"/>
@@ -13,7 +21,5 @@
       <origin xyz="0 0 0.01"/>
         <geometry>
-          <mesh filename="package://akabot_description/meshes/base_cylinder.dae"/>
-          <!-- <mesh filename="package://akabot_description/meshes/base_cylinder.stl" scale ="0.0001 0.0001 0.0001"/> -->
-          <!-- <mesh filename="file://$(find akabot_description)/meshes/base_cylinder.stl" scale ="0.0001 0.0001 0.0001"/> -->
+          <mesh filename="package://akabot_description/meshes/base_cylinder.stl" scale ="0.0001 0.0001 0.0001"/>
         </geometry>
         <material name="black">
@@ -24,19 +30,10 @@
       <origin xyz="0 0 0.01"/>
         <geometry>
-          <mesh filename="package://akabot_description/meshes/base_cylinder.dae"/>
-          <!-- <mesh filename="package://akabot_description/meshes/base_cylinder.stl" scale ="0.0001 0.0001 0.0001"/> -->
-          <!-- <mesh filename="file://$(find akabot_description)/meshes/base_cylinder.stl" scale ="0.0001 0.0001 0.0001"/> -->
+          <mesh filename="package://akabot_description/meshes/base_cylinder.stl" scale ="0.0001 0.0001 0.0001"/>
         </geometry>
     </collision>
-		<inertial>
-      <mass value="0.540142"/>
-      <inertia
-        ixx="0.0021190000"
-        iyy="0.0006925000"
-        izz="0.0025280000"
-        ixy="-0.0000172100"
-        ixz="0.0000006389"
-        iyz="0.0000461200"/>
-    </inertial>
+    <xacro:box_inertia mass="0.527" length="0.215" width="0.112" height="0.052">
+      <origin xyz="0 0 0" rpy="0 0 0"/>
+    </xacro:box_inertia>
   </link>
   <joint name="top_plate_joint" type="revolute">
@@ -52,28 +49,16 @@
       <origin xyz="0 0 0"/>
         <geometry>
-          <mesh filename="package://akabot_description/meshes/top_plate.dae"/>
-          <!-- <mesh filename="package://akabot_description/meshes/top_plate.stl" scale ="0.001 0.001 0.001"/> -->
-          <!-- <mesh filename="file://$(find akabot_description)/meshes/top_plate.stl" scale ="0.001 0.001 0.001"/> -->
+          <mesh filename="package://akabot_description/meshes/top_plate.stl" scale ="0.001 0.001 0.001"/>
         </geometry>
         <material name="black"/>
     </visual>
 	  <collision>
-      <!-- <origin xyz="0 0 0"/> -->
-      <geometry>
-        <mesh filename="package://akabot_description/meshes/top_plate.dae"/>
-        <!-- <mesh filename="package://akabot_description/meshes/top_plate.stl" scale ="0.001 0.001 0.001"/> -->
-        <!-- <mesh filename="file://$(find akabot_description)/meshes/top_plate.stl" scale ="0.001 0.001 0.001"/> -->
-      </geometry>
-    </collision>
-		<inertial>
-      <mass value="0.480879"/>
-      <inertia
-        ixx="0.0003790000"
-        iyy="0.0005557000"
-        izz="0.0005889000"
-        ixy="0.0000000022"
-        ixz="-0.0000003561"
-        iyz="0.0000012247"/>
-		</inertial>
+      <geometry>
+        <mesh filename="package://akabot_description/meshes/top_plate.stl" scale ="0.001 0.001 0.001"/>
+      </geometry>
+    </collision>
+    <xacro:cylinder_inertia mass="0.115" length="0.002" radius="0.055">
+      <origin xyz="0 0 0" rpy="0 0 0"/>
+    </xacro:cylinder_inertia>
   </link>
   <joint name="lower_arm_joint" type="revolute">
@@ -87,9 +72,6 @@
   <link name="lower_arm">
     <visual>
-      <!-- <origin xyz="0 0 0"/> -->
-      <geometry>
-        <mesh filename="package://akabot_description/meshes/lower_arm.dae"/>
-        <!-- <mesh filename="package://akabot_description/meshes/lower_arm.stl" scale ="0.001 0.001 0.001"/> -->
-        <!-- <mesh filename="file://$(find akabot_description)/meshes/lower_arm.stl" scale ="0.001 0.001 0.001"/> -->
+      <geometry>
+        <mesh filename="package://akabot_description/meshes/lower_arm.stl" scale ="0.001 0.001 0.001"/>
       </geometry>
       <material name="black"/>
@@ -98,19 +80,10 @@
       <origin xyz="0 0 0"/>
       <geometry>
-        <mesh filename="package://akabot_description/meshes/lower_arm.dae"/>
-        <!-- <mesh filename="package://akabot_description/meshes/lower_arm.stl" scale ="0.001 0.001 0.001"/> -->
-        <!-- <mesh filename="file://$(find akabot_description)/meshes/lower_arm.stl" scale ="0.001 0.001 0.001"/> -->
-      </geometry>
-    </collision>
-		<inertial>
-      <mass value="0.297781"/>
-      <inertia
-        ixx="0.0017100000"
-        iyy="0.0016310000"
-        izz="0.0001482000"
-        ixy="-0.0000011433"
-        ixz="0.0000021161"
-        iyz="0.0002135000"/>
-    </inertial>
+        <mesh filename="package://akabot_description/meshes/lower_arm.stl" scale ="0.001 0.001 0.001"/>
+      </geometry>
+    </collision>
+    <xacro:box_inertia mass="0.047" length="0.13" width="0.056" height="0.025">
+      <origin xyz="0 0 0" rpy="0 0 0"/>
+    </xacro:box_inertia>
   </link>
   <joint name="upper_arm_joint" type="revolute">
@@ -126,7 +99,5 @@
       <origin rpy="0 1.59 0" xyz="0 0 0"/>
       <geometry>
-        <mesh filename="package://akabot_description/meshes/upper_arm.dae"/>
-        <!-- <mesh filename="package://akabot_description/meshes/upper_arm.stl" scale ="0.001 0.001 0.001"/> -->
-        <!-- <mesh filename="file://$(find akabot_description)/meshes/upper_arm.stl" scale ="0.001 0.001 0.001"/> -->
+        <mesh filename="package://akabot_description/meshes/upper_arm.stl" scale ="0.001 0.001 0.001"/>
       </geometry>
       <material name="black"/>
@@ -135,13 +106,10 @@
       <origin rpy="0 1.59 0" xyz="0 0 0"/>
       <geometry>
-        <mesh filename="package://akabot_description/meshes/upper_arm.dae"/>
-        <!-- <mesh filename="package://akabot_description/meshes/upper_arm.stl" scale ="0.001 0.001 0.001"/> -->
-        <!-- <mesh filename="file://$(find akabot_description)/meshes/upper_arm.stl" scale ="0.001 0.001 0.001"/> -->
-      </geometry>
-    </collision>
-		<inertial>
-			<mass value="2e-06"/>
-			<inertia ixx="1.1e-09" ixy="0" ixz="0" iyy="1.1e-09" iyz="0" izz="1.1e-09"/>
-		</inertial>
+        <mesh filename="package://akabot_description/meshes/upper_arm.stl" scale ="0.001 0.001 0.001"/>
+      </geometry>
+    </collision>
+    <xacro:box_inertia mass="0.105" length="0.185" width="0.036" height="0.025">
+      <origin xyz="0 0 0" rpy="0 0 0"/>
+    </xacro:box_inertia>
   </link>
   <joint name="wrist_joint" type="revolute">
@@ -155,9 +123,6 @@
   <link name="wrist">
     <visual>
-      <!-- <origin rpy="0 0 0" xyz="0 0 0"/> -->
-      <geometry>
-        <mesh filename="package://akabot_description/meshes/wrist.dae"/>
-        <!-- <mesh filename="package://akabot_description/meshes/wrist.stl" scale ="0.001 0.001 0.001"/> -->
-        <!-- <mesh filename="file://$(find akabot_description)/meshes/wrist.stl" scale ="0.001 0.001 0.001"/> -->
+      <geometry>
+        <mesh filename="package://akabot_description/meshes/wrist.stl" scale ="0.001 0.001 0.001"/>
       </geometry>
       <material name="black"/>
@@ -166,19 +131,10 @@
       <origin rpy="0 0 0" xyz="0 0 0"/>
       <geometry>
-        <mesh filename="package://akabot_description/meshes/wrist.dae"/>
-        <!-- <mesh filename="package://akabot_description/meshes/wrist.stl" scale ="0.001 0.001 0.001"/> -->
-        <!-- <mesh filename="file://$(find akabot_description)/meshes/wrist.stl" scale ="0.001 0.001 0.001"/> -->
-      </geometry>
-    </collision>
-		<inertial>
-      <mass value="0.283651"/>
-      <inertia
-        ixx="0.0011850000"
-        iyy="0.0000682900"
-        izz="0.0012060000"
-        ixy="-0.0000024317"
-        ixz="0.0000000000"
-        iyz="0.0000000000"/>
-    </inertial>
+        <mesh filename="package://akabot_description/meshes/wrist.stl" scale ="0.001 0.001 0.001"/>
+      </geometry>
+    </collision>
+    <xacro:box_inertia mass="0.082" length="0.065" width="0.057" height="0.025">
+      <origin xyz="0 0 0" rpy="0 0 0"/>
+    </xacro:box_inertia>
   </link>
   <joint name="claw_base_joint" type="revolute">
@@ -194,7 +150,5 @@
       <origin rpy="0 3.18 0" xyz="0 0 0"/>
       <geometry>
-        <mesh filename="package://akabot_description/meshes/claw_base.dae"/>
-        <!-- <mesh filename="package://akabot_description/meshes/claw_base.stl" scale ="0.001 0.001 0.001"/> -->
-        <!-- <mesh filename="file://$(find akabot_description)/meshes/claw_base.stl" scale ="0.001 0.001 0.001"/> -->
+        <mesh filename="package://akabot_description/meshes/claw_base.stl" scale ="0.001 0.001 0.001"/>
       </geometry>
       <material name="white">
@@ -205,24 +159,15 @@
       <origin rpy="0 3.18 0" xyz="0 0 0"/>
       <geometry>
-        <mesh filename="package://akabot_description/meshes/claw_base.dae"/>
-        <!-- <mesh filename="package://akabot_description/meshes/claw_base.stl" scale ="0.001 0.001 0.001"/> -->
-        <!-- <mesh filename="file://$(find akabot_description)/meshes/claw_base.stl" scale ="0.001 0.001 0.001"/> -->
-      </geometry>
-    </collision>
-		<inertial>
-     <mass value="0.084957"/>
-      <inertia
-        ixx="0.0000308200"
-        iyy="0.0000282200"
-        izz="0.0000315200"
-        ixy="0.0000000191"
-        ixz="0.0000000023"
-        iyz="0.0000025481"/>
-    </inertial>
+        <mesh filename="package://akabot_description/meshes/claw_base.stl" scale ="0.001 0.001 0.001"/>
+      </geometry>
+    </collision>
+    <xacro:box_inertia mass="0.079" length="0.07" width="0.05" height="0.015">
+      <origin xyz="0 0 0" rpy="0 0 0"/>
+    </xacro:box_inertia>
   </link>
   <joint name="right_claw_joint" type="revolute">
     <parent link="claw_base"/>
     <child link="right_claw"/>
-    <origin rpy="0 0 -0.31" xyz="0.11 0.34 0"/>
+    <origin rpy="0 0 -0.31" xyz="0.11 0.335 0.0155"/>
     <axis xyz="0 0 1" />
     <limit effort="1000.0" lower="-0.5" upper="0.0" velocity="1.0" />
@@ -233,7 +178,5 @@
       <origin rpy="0 0 0" xyz="0 0 0"/>
       <geometry>
-        <mesh filename="package://akabot_description/meshes/right_claw.dae"/>
-        <!-- <mesh filename="package://akabot_description/meshes/right_claw.stl" scale ="0.001 0.001 0.001"/> -->
-        <!-- <mesh filename="file://$(find akabot_description)/meshes/right_claw.stl" scale ="0.001 0.001 0.001"/> -->
+        <mesh filename="package://akabot_description/meshes/right_claw.stl" scale ="0.001 0.001 0.001"/>
       </geometry>
       <material name="white"/>
@@ -242,19 +185,10 @@
       <origin rpy="0 0 0" xyz="0 0 0"/>
       <geometry>
-        <mesh filename="package://akabot_description/meshes/right_claw.dae"/>
-        <!-- <mesh filename="package://akabot_description/meshes/right_claw.stl" scale ="0.001 0.001 0.001"/> -->
-        <!-- <mesh filename="file://$(find akabot_description)/meshes/right_claw.stl" scale ="0.001 0.001 0.001"/> -->
-      </geometry>
-    </collision>
-		<inertial>
-      <mass value="0.072885"/>
-      <inertia
-        ixx="0.0000253700"
-        iyy="0.0000183600"
-        izz="0.0000167400"
-        ixy="0.0000000000"
-        ixz="0.0000000000"
-        iyz="0.0000004340"/>
-      </inertial>
+        <mesh filename="package://akabot_description/meshes/right_claw.stl" scale ="0.001 0.001 0.001"/>
+      </geometry>
+    </collision>
+    <xacro:box_inertia mass="0.019" length="0.1" width="0.01" height="0.012">
+      <origin xyz="0 0 0" rpy="0 0 0"/>
+    </xacro:box_inertia>
   </link>
   <!-- Left claw -->
@@ -263,7 +197,5 @@
       <origin rpy="0 0 0" xyz="0 0 0"/>
       <geometry>
-        <mesh filename="package://akabot_description/meshes/left_claw.dae"/>
-        <!-- <mesh filename="package://akabot_description/meshes/left_claw.stl" scale ="0.001 0.001 0.001"/> -->
-        <!-- <mesh filename="file://$(find akabot_description)/meshes/left_claw.stl" scale ="0.001 0.001 0.001"/> -->
+        <mesh filename="package://akabot_description/meshes/left_claw.stl" scale ="0.001 0.001 0.001"/>
       </geometry>
       <material name="white"/>
@@ -272,19 +204,10 @@
       <origin rpy="0 0 0" xyz="0 0 0"/>
       <geometry>
-        <mesh filename="package://akabot_description/meshes/left_claw.dae"/>
-        <!-- <mesh filename="package://akabot_description/meshes/left_claw.stl" scale ="0.001 0.001 0.001"/> -->
-        <!-- <mesh filename="file://$(find akabot_description)/meshes/left_claw.stl" scale ="0.001 0.001 0.001"/> -->
-      </geometry>
-    </collision>
-		<inertial>
-      <mass value="0.072885"/>
-      <inertia
-        ixx="0.0000253700"
-        iyy="0.0000183600"
-        izz="0.0000167400"
-        ixy="0.0000000000"
-        ixz="0.0000000000"
-        iyz="0.0000004340"/>
-    </inertial>
+        <mesh filename="package://akabot_description/meshes/left_claw.stl" scale ="0.001 0.001 0.001"/>
+      </geometry>
+    </collision>
+    <xacro:box_inertia mass="0.019" length="0.1" width="0.01" height="0.012">
+      <origin xyz="0 0 0" rpy="0 0 0"/>
+    </xacro:box_inertia>
   </link>
   <joint name="left_claw_joint" type="revolute">

Commit message: Correctly resize akabot model

File: akabot_description/urdf/akabot_core.xacro (robot description, xacro)
@@ -19,7 +19,7 @@
   <link name="base_plate">
     <visual>
-      <origin xyz="0 0 0.01"/>
+      <origin xyz="0 0 0.001"/>
         <geometry>
-          <mesh filename="package://akabot_description/meshes/base_cylinder.stl" scale ="0.0001 0.0001 0.0001"/>
+          <mesh filename="package://akabot_description/meshes/base_cylinder.stl" scale ="0.00001 0.00001 0.00001"/>
         </geometry>
         <material name="black">
@@ -28,7 +28,7 @@
     </visual>
 	  <collision>
-      <origin xyz="0 0 0.01"/>
+      <origin xyz="0 0 0.001"/>
         <geometry>
-          <mesh filename="package://akabot_description/meshes/base_cylinder.stl" scale ="0.0001 0.0001 0.0001"/>
+          <mesh filename="package://akabot_description/meshes/base_cylinder.stl" scale ="0.00001 0.00001 0.00001"/>
         </geometry>
     </collision>
@@ -40,5 +40,5 @@
     <parent link="base_plate"/>
     <child link="top_plate"/>
-    <origin rpy="0 0 1.5" xyz="0 0 0.48"/>
+    <origin rpy="0 0 1.5" xyz="0 0 0.048"/>
     <axis xyz="0 0 1" />
     <limit effort="1000.0" lower="1.56" upper="4.68" velocity="1.0" />
@@ -49,5 +49,5 @@
       <origin xyz="0 0 0"/>
         <geometry>
-          <mesh filename="package://akabot_description/meshes/top_plate.stl" scale ="0.001 0.001 0.001"/>
+          <mesh filename="package://akabot_description/meshes/top_plate.stl" scale ="0.0001 0.0001 0.0001"/>
         </geometry>
         <material name="black"/>
@@ -55,5 +55,5 @@
 	  <collision>
       <geometry>
-        <mesh filename="package://akabot_description/meshes/top_plate.stl" scale ="0.001 0.001 0.001"/>
+        <mesh filename="package://akabot_description/meshes/top_plate.stl" scale ="0.0001 0.0001 0.0001"/>
       </geometry>
     </collision>
@@ -65,5 +65,5 @@
     <parent link="top_plate"/>
     <child link="lower_arm"/>
-    <origin xyz="0 0.19 0.28"/>
+    <origin xyz="0 0.019 0.028"/>
     <axis xyz="1 0 0" />
     <limit effort="1000.0" lower="0.0" upper="3.12" velocity="1.0" />
@@ -73,5 +73,5 @@
     <visual>
       <geometry>
-        <mesh filename="package://akabot_description/meshes/lower_arm.stl" scale ="0.001 0.001 0.001"/>
+        <mesh filename="package://akabot_description/meshes/lower_arm.stl" scale ="0.0001 0.0001 0.0001"/>
       </geometry>
       <material name="black"/>
@@ -80,5 +80,5 @@
       <origin xyz="0 0 0"/>
       <geometry>
-        <mesh filename="package://akabot_description/meshes/lower_arm.stl" scale ="0.001 0.001 0.001"/>
+        <mesh filename="package://akabot_description/meshes/lower_arm.stl" scale ="0.0001 0.0001 0.0001"/>
       </geometry>
     </collision>
@@ -90,5 +90,5 @@
     <parent link="lower_arm"/>
     <child link="upper_arm"/>
-    <origin xyz="-0.25 1.0 0"/>
+    <origin xyz="-0.025 0.1 0"/>
     <axis xyz="1 0 0" />
     <limit effort="1000.0" lower="-1.7" upper="1.7" velocity="1.0" />
@@ -99,5 +99,5 @@
       <origin rpy="0 1.59 0" xyz="0 0 0"/>
       <geometry>
-        <mesh filename="package://akabot_description/meshes/upper_arm.stl" scale ="0.001 0.001 0.001"/>
+        <mesh filename="package://akabot_description/meshes/upper_arm.stl" scale ="0.0001 0.0001 0.0001"/>
       </geometry>
       <material name="black"/>
@@ -106,5 +106,5 @@
       <origin rpy="0 1.59 0" xyz="0 0 0"/>
       <geometry>
-        <mesh filename="package://akabot_description/meshes/upper_arm.stl" scale ="0.001 0.001 0.001"/>
+        <mesh filename="package://akabot_description/meshes/upper_arm.stl" scale ="0.0001 0.0001 0.0001"/>
       </geometry>
     </collision>
@@ -116,5 +116,5 @@
     <parent link="upper_arm"/>
     <child link="wrist"/>
-    <origin xyz="0.11 1.25 0"/>
+    <origin xyz="0.011 0.125 0"/>
     <axis xyz="1 0 0" />
     <limit effort="1000.0" lower="-1.7" upper="1.7" velocity="1.0" />
@@ -124,5 +124,5 @@
     <visual>
       <geometry>
-        <mesh filename="package://akabot_description/meshes/wrist.stl" scale ="0.001 0.001 0.001"/>
+        <mesh filename="package://akabot_description/meshes/wrist.stl" scale ="0.0001 0.0001 0.0001"/>
       </geometry>
       <material name="black"/>
@@ -131,5 +131,5 @@
       <origin rpy="0 0 0" xyz="0 0 0"/>
       <geometry>
-        <mesh filename="package://akabot_description/meshes/wrist.stl" scale ="0.001 0.001 0.001"/>
+        <mesh filename="package://akabot_description/meshes/wrist.stl" scale ="0.0001 0.0001 0.0001"/>
       </geometry>
     </collision>
@@ -143,5 +143,5 @@
     <parent link="wrist"/>
     <child link="claw_base"/>
-    <origin xyz="0 0.63 0"/>
+    <origin xyz="0 0.063 0"/>
   </joint>
   <!-- Claw base -->
@@ -150,5 +150,5 @@
       <origin rpy="0 3.18 0" xyz="0 0 0"/>
       <geometry>
-        <mesh filename="package://akabot_description/meshes/claw_base.stl" scale ="0.001 0.001 0.001"/>
+        <mesh filename="package://akabot_description/meshes/claw_base.stl" scale ="0.0001 0.0001 0.0001"/>
       </geometry>
       <material name="white">
@@ -159,5 +159,5 @@
       <origin rpy="0 3.18 0" xyz="0 0 0"/>
       <geometry>
-        <mesh filename="package://akabot_description/meshes/claw_base.stl" scale ="0.001 0.001 0.001"/>
+        <mesh filename="package://akabot_description/meshes/claw_base.stl" scale ="0.0001 0.0001 0.0001"/>
       </geometry>
     </collision>
@@ -169,5 +169,5 @@
     <parent link="claw_base"/>
     <child link="right_claw"/>
-    <origin rpy="0 0 -0.31" xyz="0.11 0.335 0.0155"/>
+    <origin rpy="0 0 -0.31" xyz="0.011 0.0335 0.00155"/>
     <axis xyz="0 0 1" />
     <limit effort="1000.0" lower="-0.5" upper="0.0" velocity="1.0" />
@@ -178,5 +178,5 @@
       <origin rpy="0 0 0" xyz="0 0 0"/>
       <geometry>
-        <mesh filename="package://akabot_description/meshes/right_claw.stl" scale ="0.001 0.001 0.001"/>
+        <mesh filename="package://akabot_description/meshes/right_claw.stl" scale ="0.0001 0.0001 0.0001"/>
       </geometry>
       <material name="white"/>
@@ -185,5 +185,5 @@
       <origin rpy="0 0 0" xyz="0 0 0"/>
       <geometry>
-        <mesh filename="package://akabot_description/meshes/right_claw.stl" scale ="0.001 0.001 0.001"/>
+        <mesh filename="package://akabot_description/meshes/right_claw.stl" scale ="0.0001 0.0001 0.0001"/>
       </geometry>
     </collision>
@@ -197,5 +197,5 @@
       <origin rpy="0 0 0" xyz="0 0 0"/>
       <geometry>
-        <mesh filename="package://akabot_description/meshes/left_claw.stl" scale ="0.001 0.001 0.001"/>
+        <mesh filename="package://akabot_description/meshes/left_claw.stl" scale ="0.0001 0.0001 0.0001"/>
       </geometry>
       <material name="white"/>
@@ -204,5 +204,5 @@
       <origin rpy="0 0 0" xyz="0 0 0"/>
       <geometry>
-        <mesh filename="package://akabot_description/meshes/left_claw.stl" scale ="0.001 0.001 0.001"/>
+        <mesh filename="package://akabot_description/meshes/left_claw.stl" scale ="0.0001 0.0001 0.0001"/>
       </geometry>
     </collision>
@@ -214,5 +214,5 @@
     <parent link="claw_base"/>
     <child link="left_claw"/>
-    <origin rpy="0 0 0.22" xyz="-0.16 0.30 0"/>
+    <origin rpy="0 0 0.22" xyz="-0.016 0.030 0"/>
     <axis xyz="0 0 1" />
     <limit effort="1000.0" lower="0.0" upper="0.5" velocity="1.0" />

File: akabot_description/urdf/depth_camera.xacro (robot description, xacro)
@@ -3,13 +3,13 @@
   <link name="camera_link">
     <visual>
-      <origin xyz="0.4 -0.015 0.135" rpy="${-pi/2} ${pi} ${-pi/2}"/>
+      <origin xyz="0.04 -0.0015 0.0135" rpy="${-pi/2} ${pi} ${-pi/2}"/>
         <geometry>
-          <mesh filename="package://akabot_description/meshes/d415.dae" scale="10 10 10"/>
+          <mesh filename="package://akabot_description/meshes/d415.dae"/>
         </geometry>
     </visual>
     <collision>
-      <origin xyz="0.4 -0.015 0.135" rpy="${-pi/2} ${pi} ${-pi/2}"/>
+      <origin xyz="0.04 -0.0015 0.0135" rpy="${-pi/2} ${pi} ${-pi/2}"/>
         <geometry>
-          <mesh filename="package://akabot_description/meshes/d415.dae" scale="10 10 10"/>
+          <mesh filename="package://akabot_description/meshes/d415.dae"/>
         </geometry>
     </collision>
@@ -18,5 +18,5 @@
     <parent link="base_plate"/>
     <child link="camera_link"/>
-    <origin xyz="0.205 0 0.0425" rpy="0 0 0"/>
+    <origin xyz="0.0205 0 0.00425" rpy="0 0 0"/>
   </joint>
   <link name="camera_link_optical"></link>

Commit message: Create pick and place Gazebo classic world

File: akabot_description/urdf/akabot_core.xacro (robot description, xacro)
@@ -44,4 +44,8 @@
     <limit effort="1000.0" lower="1.56" upper="4.68" velocity="1.0" />
   </joint>
+  <gazebo reference="base_plate">
+    <mu1 value="1.16"/>
+    <mu2 value="1.16"/>
+  </gazebo>
   <!-- Top plate -->
   <link name="top_plate">

File: akabot_description/urdf/depth_camera.xacro (robot description, xacro)
@@ -1,4 +1,5 @@
 <?xml version="1.0" ?>
 <robot xmlns:xacro="http://ros.org/wiki/xacro">
+  <!-- Intel RealSense D415 camera -->
   <link name="camera_link">
     <visual>
@@ -26,4 +27,5 @@
     <origin xyz="0 0 0" rpy="${-pi/2} 0 ${-pi/2}"/>
   </joint>
+  <xacro:property name="deg_to_rad" value="0.01745329252" />
   <gazebo reference="camera_link">
     <sensor name="camera" type="depth">
@@ -32,9 +34,9 @@
         <update_rate>10</update_rate>
         <camera>
-          <horizontal_fov>1.2113</horizontal_fov>
+        <horizontal_fov>${69.4*deg_to_rad}</horizontal_fov>
           <image>
             <format>B8G8R8</format>
-            <width>1280</width>
-            <height>720</height>
+            <width>640</width>
+            <height>480</height>
           </image>
           <clip>
