Commit message: Update moveit_config package

File: akabot_moveit_config/config/akabot.ros2_control.xacro (robot description, xacro)
@@ -8,11 +8,4 @@
                 <plugin>mock_components/GenericSystem</plugin>
             </hardware>
-            <joint name="claw_base_joint">
-                <command_interface name="position"/>
-                <state_interface name="position">
-                  <param name="initial_value">${initial_positions['claw_base_joint']}</param>
-                </state_interface>
-                <state_interface name="velocity"/>
-            </joint>
             <joint name="right_claw_joint">
                 <command_interface name="position"/>
@@ -50,4 +43,11 @@
                 <state_interface name="velocity"/>
             </joint>
+            <joint name="claw_base_joint">
+                <command_interface name="position"/>
+                <state_interface name="position">
+                  <param name="initial_value">${initial_positions['claw_base_joint']}</param>
+                </state_interface>
+                <state_interface name="velocity"/>
+            </joint>
         </ros2_control>
     </xacro:macro>
